Commit message: Update robot_arm.xacro

File: robot_arm.xacro (robot description, xacro)
@@ -16,4 +16,5 @@
         <mesh filename="file:///home/mikepzaza/Desktop/project2/src/articubot_two/A1V2.dae" scale="1 1 1"/>
       </geometry>
+      <material name="yellow"/>
     </visual>
     <collision>
@@ -27,5 +28,5 @@
     </link>
     <gazebo reference="link_8">
-    <material>Gazebo/White</material>
+    <material>Gazebo/Yellow</material>
     </gazebo>
   <!-- Joint between link_8 and link_9 -->
@@ -43,4 +44,5 @@
         <mesh filename="file:///home/mikepzaza/Desktop/project2/src/articubot_two/A2.dae" scale="1 1 1"/>
       </geometry>
+      <material name="yellow"/>
     </visual>
     <collision>
@@ -54,5 +56,5 @@
   </link>
     <gazebo reference="link_9">
-    <material>Gazebo/White</material>
+    <material>Gazebo/Yellow</material>
     </gazebo>
   <!-- Joint between link_9 and link_10 -->
@@ -71,4 +73,5 @@
         <mesh filename="file:///home/mikepzaza/Desktop/project2/src/articubot_two/A3.dae" scale="1 1 1"/>
       </geometry>
+      <material name="yellow"/>
     </visual>
     <collision>
@@ -82,5 +85,5 @@
   </link>
     <gazebo reference="link_10">
-    <material>Gazebo/White</material>
+    <material>Gazebo/Yellow</material>
     </gazebo>
 </robot>
