Commit message: Update robot_core.xacro

File: robot_core.xacro (robot description, xacro)
@@ -49,13 +49,13 @@
     <visual>
       <geometry>
+        <mesh filename="/home/mikepzaza/Desktop/project2/src/articubot_two/T1V2.dae" scale="1 1 1"/>
+      </geometry>
+    </visual>
+    <collision>
+      <geometry>
         <mesh filename="/home/mikepzaza/Desktop/project2/src/articubot_two/T1.dae" scale="1 1 1"/>
       </geometry>
-    </visual>
-    <collision>
-      <geometry>
-        <mesh filename="/home/mikepzaza/Desktop/project2/src/articubot_two/T1.dae" scale="1 1 1"/>
-      </geometry>
-    </collision>
-    <xacro:inertial_box mass="0.1" x="0.005" y="0.140" z="0.08">
+    </collision>
+    <xacro:inertial_box mass="0.1" x="0.005" y="0.14" z="0.08">
         <origin xyz="0 0 0" rpy="0 0 0"/>
     </xacro:inertial_box>
@@ -68,5 +68,5 @@
     <parent link="base_link"/>
     <child link="link_1"/>
-    <origin xyz="0.071711 0.055977 0.02748" rpy="0 0 0"/>
+    <origin xyz="0.073 0.05597 0.02748" rpy="0 0 0"/>
     <axis xyz="1 0 0"/>
     <limit effort="5.0" velocity="1.0" lower="-0.540" upper="0.540"/>
@@ -76,13 +76,13 @@
     <visual>
       <geometry>
-        <mesh filename="/home/mikepzaza/Desktop/project2/src/articubot_two/T2.dae" scale="1 1 1"/>
-      </geometry>
-    </visual>
-    <collision>
-      <geometry>
-        <mesh filename="/home/mikepzaza/Desktop/project2/src/articubot_two/T2.dae" scale="1 1 1"/>
-      </geometry>
-    </collision>
-    <xacro:inertial_box mass="0.1" x="0.005" y="0.140" z="0.08">
+        <mesh filename="/home/mikepzaza/Desktop/project2/src/articubot_two/T2V2.dae" scale="1 1 1"/>
+      </geometry>
+    </visual>
+    <collision>
+      <geometry>
+        <mesh filename="/home/mikepzaza/Desktop/project2/src/articubot_two/T2V2.dae" scale="1 1 1"/>
+      </geometry>
+    </collision>
+    <xacro:inertial_box mass="0.1" x="0.005" y="0.14" z="0.08">
         <origin xyz="0 0 0" rpy="0 0 0"/>
     </xacro:inertial_box>
@@ -103,5 +103,5 @@
     <visual>
       <geometry>
-        <mesh filename="/home/mikepzaza/Desktop/project2/src/articubot_two/Wh1.dae" scale="1 1 1"/>
+        <mesh filename="/home/mikepzaza/Desktop/project2/src/articubot_two/W1V2.dae" scale="1 1 1"/>
       </geometry>
     </visual>
@@ -122,5 +122,5 @@
     <parent link="base_link"/>
     <child link="link_6"/>
-    <origin xyz="-0.311289 -0.214023 -0.03252" rpy="0 0 0"/>
+    <origin xyz="-0.312 -0.214023 -0.03252" rpy="0 0 0"/>
     <axis xyz="1 0 0"/>
   </joint>
@@ -146,7 +146,7 @@
   <!-- Joint between base_link and link_6_clone -->
   <joint name="joint_6_clone" type="continuous">
-    <parent link="base_link"/>
+    <parent link="link_2"/>
     <child link="link_6_clone"/>
-    <origin xyz="-0.309489 -0.014223 -0.03352" rpy="0 0 0"/>
+    <origin xyz="-0.034 -0.07 -0.06" rpy="0 0 0"/>
     <axis xyz="1 0 0"/>
   </joint>
@@ -172,7 +172,7 @@
   <!-- Joint between link_6_clone and link_6_clone_clone -->
   <joint name="joint_6_clone_clone" type="continuous">
-    <parent link="base_link"/>
+    <parent link="link_2"/>
     <child link="link_6_clone_clone"/>
-    <origin xyz="-0.310175 0.126662 -0.032377" rpy="0 0 0"/>
+    <origin xyz="-0.034 0.07 -0.06" rpy="0 0 0"/>
     <axis xyz="1 0 0"/>
   </joint>
@@ -181,5 +181,5 @@
     <visual>
       <geometry>
-        <mesh filename="/home/mikepzaza/Desktop/project2/src/articubot_two/W2.dae" scale="1 1 1"/>
+        <mesh filename="/home/mikepzaza/Desktop/project2/src/articubot_two/W2V2.dae" scale="1 1 1"/>
       </geometry>
     </visual>
@@ -200,5 +200,5 @@
     <parent link="base_link"/>
     <child link="link_7"/>
-    <origin xyz="0.105211 -0.213773 -0.03252" rpy="0 0 0"/>
+    <origin xyz="0.106 -0.213773 -0.03252" rpy="0 0 0"/>
     <axis xyz="1 0 0"/>
   </joint>
@@ -224,7 +224,7 @@
   <!-- Joint between link_7 and link_7_clone -->
   <joint name="joint_7_clone" type="continuous">
-    <parent link="base_link"/>
+    <parent link="link_1"/>
     <child link="link_7_clone"/>
-    <origin xyz="0.103627 -0.014982 -0.032687" rpy="0 0 0"/>
+    <origin xyz="0.035 -0.07 -0.06" rpy="0 0 0"/>
     <axis xyz="1 0 0"/>
   </joint>
@@ -250,7 +250,7 @@
   <!-- Joint between link_7_clone and link_7_clone_clone -->
   <joint name="joint_7_clone_clone" type="continuous">
-    <parent link="base_link"/>
+    <parent link="link_1"/>
     <child link="link_7_clone_clone"/>
-    <origin xyz="0.102638 0.124888 -0.032691" rpy="0 0 0"/>
+    <origin xyz="0.035 0.07 -0.06" rpy="0 0 0"/>
     <axis xyz="1 0 0"/>
   </joint>

Commit message: Update robot_core.xacro

File: robot_core.xacro (robot description, xacro)
@@ -18,5 +18,4 @@
     <!-- BASE LINK -->
     <link name="base_link">
-    <origin xyz="0 0 0" rpy="0 0 0"/>
     </link>
   <!-- Link 0(baselink) -->
@@ -32,5 +31,5 @@
       </geometry>
     </collision>
-    <xacro:inertial_box mass="1.5" x="0.480" y="0.510" z="0.33">
+    <xacro:inertial_box mass="4" x="0.480" y="0.510" z="0.33">
         <origin xyz="0 0 0" rpy="0 0 0"/>
     </xacro:inertial_box>
@@ -57,5 +56,5 @@
       </geometry>
     </collision>
-    <xacro:inertial_box mass="0.1" x="0.005" y="0.14" z="0.08">
+    <xacro:inertial_box mass="0.8" x="0.005" y="0.14" z="0.08">
         <origin xyz="0 0 0" rpy="0 0 0"/>
     </xacro:inertial_box>
@@ -84,5 +83,5 @@
       </geometry>
     </collision>
-    <xacro:inertial_box mass="0.1" x="0.005" y="0.14" z="0.08">
+    <xacro:inertial_box mass="0.8" x="0.005" y="0.14" z="0.08">
         <origin xyz="0 0 0" rpy="0 0 0"/>
     </xacro:inertial_box>
@@ -111,5 +110,5 @@
       </geometry>
     </collision>
-    <xacro:inertial_cylinder mass="0.15" length="0.06" radius="0.06">
+    <xacro:inertial_cylinder mass="0.3" length="0.06" radius="0.06">
         <origin xyz="0 0 0" rpy="0 0 0"/>
     </xacro:inertial_cylinder>
@@ -129,13 +128,13 @@
     <visual>
       <geometry>
-        <mesh filename="/home/mikepzaza/Desktop/project2/src/articubot_two/Wh1.dae" scale="1 1 1"/>
-      </geometry>
-    </visual>
-    <collision>
-      <geometry>
-          <cylinder radius="0.06" length="0.06"/>
-      </geometry>
-    </collision>
-    <xacro:inertial_cylinder mass="0.15" length="0.06" radius="0.06">
+        <mesh filename="/home/mikepzaza/Desktop/project2/src/articubot_two/W1V2.dae" scale="1 1 1"/>
+      </geometry>
+    </visual>
+    <collision>
+      <geometry>
+          <cylinder radius="0.06" length="0.06"/>
+      </geometry>
+    </collision>
+    <xacro:inertial_cylinder mass="0.3" length="0.06" radius="0.06">
         <origin xyz="0 0 0" rpy="0 0 0"/>
     </xacro:inertial_cylinder>
@@ -155,13 +154,13 @@
     <visual>
       <geometry>
-        <mesh filename="/home/mikepzaza/Desktop/project2/src/articubot_two/Wh1.dae" scale="1 1 1"/>
-      </geometry>
-    </visual>
-    <collision>
-      <geometry>
-          <cylinder radius="0.06" length="0.06"/>
-      </geometry>
-    </collision>
-    <xacro:inertial_cylinder mass="0.15" length="0.06" radius="0.06">
+        <mesh filename="/home/mikepzaza/Desktop/project2/src/articubot_two/W1V2.dae" scale="1 1 1"/>
+      </geometry>
+    </visual>
+    <collision>
+      <geometry>
+          <cylinder radius="0.06" length="0.06"/>
+      </geometry>
+    </collision>
+    <xacro:inertial_cylinder mass="0.3" length="0.06" radius="0.06">
         <origin xyz="0 0 0" rpy="0 0 0"/>
     </xacro:inertial_cylinder>
@@ -189,5 +188,5 @@
       </geometry>
     </collision>
-    <xacro:inertial_cylinder mass="0.15" length="0.06" radius="0.06">
+    <xacro:inertial_cylinder mass="0.3" length="0.06" radius="0.06">
         <origin xyz="0 0 0" rpy="0 0 0"/>
     </xacro:inertial_cylinder>
@@ -207,13 +206,13 @@
     <visual>
       <geometry>
-        <mesh filename="/home/mikepzaza/Desktop/project2/src/articubot_two/W2.dae" scale="1 1 1"/>
-      </geometry>
-    </visual>
-    <collision>
-      <geometry>
-          <cylinder radius="0.06" length="0.06"/>
-      </geometry>
-    </collision>
-    <xacro:inertial_cylinder mass="0.15" length="0.06" radius="0.06">
+        <mesh filename="/home/mikepzaza/Desktop/project2/src/articubot_two/W2V2.dae" scale="1 1 1"/>
+      </geometry>
+    </visual>
+    <collision>
+      <geometry>
+          <cylinder radius="0.06" length="0.06"/>
+      </geometry>
+    </collision>
+    <xacro:inertial_cylinder mass="0.3" length="0.06" radius="0.06">
         <origin xyz="0 0 0" rpy="0 0 0"/>
     </xacro:inertial_cylinder>
@@ -233,13 +232,13 @@
     <visual>
       <geometry>
-        <mesh filename="/home/mikepzaza/Desktop/project2/src/articubot_two/W2.dae" scale="1 1 1"/>
-      </geometry>
-    </visual>
-    <collision>
-      <geometry>
-          <cylinder radius="0.06" length="0.06"/>
-      </geometry>
-    </collision>
-    <xacro:inertial_cylinder mass="0.15" length="0.06" radius="0.06">
+        <mesh filename="/home/mikepzaza/Desktop/project2/src/articubot_two/W2V2.dae" scale="1 1 1"/>
+      </geometry>
+    </visual>
+    <collision>
+      <geometry>
+          <cylinder radius="0.06" length="0.06"/>
+      </geometry>
+    </collision>
+    <xacro:inertial_cylinder mass="0.3" length="0.06" radius="0.06">
         <origin xyz="0 0 0" rpy="0 0 0"/>
     </xacro:inertial_cylinder>
@@ -267,5 +266,5 @@
       </geometry>
     </collision>
-    <xacro:inertial_box mass="0.1" x="0.015" y="0.085" z="0.05">
+    <xacro:inertial_box mass="0.4" x="0.015" y="0.085" z="0.05">
         <origin xyz="0 0 0" rpy="0 0 0"/>
     </xacro:inertial_box>
@@ -294,5 +293,5 @@
       </geometry>
     </collision>
-    <xacro:inertial_box mass="0.125" x="0.015" y="0.180" z="0.1">
+    <xacro:inertial_box mass="0.3" x="0.015" y="0.180" z="0.1">
         <origin xyz="0 0 0" rpy="0 0 0"/>
     </xacro:inertial_box>
@@ -321,5 +320,5 @@
       </geometry>
     </collision>
-    <xacro:inertial_box mass="0.1" x="0.015" y="0.180" z="0.1">
+    <xacro:inertial_box mass="0.2" x="0.015" y="0.180" z="0.1">
         <origin xyz="0 0 0" rpy="0 0 0"/>
     </xacro:inertial_box>
