Commit message: Update robot_core.xacro

File: robot_core.xacro (robot description, xacro)
@@ -1,4 +1,5 @@
 <?xml version="1.0"?>
-<robot name="botpj2v1" xmlns:xacro="http://ros.org/wiki/xacro">
+<robot xmlns:xacro="http://www.ros.org/wiki/xacro" >
+<xacro:include filename="inertial_macros.xacro" />
     <material name="white">
         <color rgba="1 1 1 1" />
@@ -16,17 +17,31 @@
      <color rgba="1 0 0 1"/>
  </material>
-    <!-- BASE LINK -->
-    <link name="base_link">
-    </link>
+  <!-- BASE LINK -->
+  <link name="base_link">
+  </link>
+  <!-- BASE_FOOTPRINT LINK -->
+  <joint name="base_footprint_joint" type="fixed">
+    <parent link="base_link"/>
+    <child link="base_footprint"/>
+    <origin xyz="0 0 0" rpy="0 0 0"/>
+  </joint>
+  <link name="base_footprint">
+  </link>
+  <!-- Joint between base_link and link_0  -->
+  <joint name="joint_0" type="fixed">
+    <parent link="base_link"/>
+    <child link="link_0"/>
+    <origin xyz="0 0 0" rpy="0 0 0"/>
+  </joint>
   <!-- Link 0(baselink) -->
   <link name="link_0">
     <visual>
       <geometry>
-        <mesh filename="/home/mikepzaza/Desktop/project2/src/articubot_two/baselink.dae" scale="1 1 1"/>
-      </geometry>
-    </visual>
-    <collision>
-      <geometry>
-        <mesh filename="/home/mikepzaza/Desktop/project2/src/articubot_two/baselink.dae" scale="1 1 1"/>
+        <mesh filename="file:///home/mikepzaza/Desktop/project2/src/articubot_two/baselink.dae" scale="1 1 1"/>
+      </geometry>
+    </visual>
+    <collision>
+      <geometry>
+        <mesh filename="file:///home/mikepzaza/Desktop/project2/src/articubot_two/baselink.dae" scale="1 1 1"/>
       </geometry>
     </collision>
@@ -38,9 +53,11 @@
     <material>Gazebo/White</material>
     </gazebo>
-  <!-- Joint between base_link and link_0  -->
-  <joint name="joint_0" type="fixed">
-    <parent link="base_link"/>
-    <child link="link_0"/>
-    <origin xyz="-0.097289 -0.049023 -0.03252" rpy="0 0 0"/>
+  <!-- Joint between link_0 and base_link -->
+  <joint name="joint_1" type="revolute">
+    <parent link="base_link"/>
+    <child link="link_1"/>
+    <origin xyz="0.170 0.08 0.06" rpy="0 0 0"/>
+    <axis xyz="1 0 0"/>
+    <limit effort="5.0" velocity="1.0" lower="-0.540" upper="0.540"/>
   </joint>
   <!-- Link 1 (T1)-->
@@ -48,10 +65,10 @@
     <visual>
       <geometry>
-        <mesh filename="/home/mikepzaza/Desktop/project2/src/articubot_two/T1V2.dae" scale="1 1 1"/>
-      </geometry>
-    </visual>
-    <collision>
-      <geometry>
-        <mesh filename="/home/mikepzaza/Desktop/project2/src/articubot_two/T1.dae" scale="1 1 1"/>
+        <mesh filename="file:///home/mikepzaza/Desktop/project2/src/articubot_two/T1V2.dae" scale="1 1 1"/>
+      </geometry>
+    </visual>
+    <collision>
+      <geometry>
+        <mesh filename="file:///home/mikepzaza/Desktop/project2/src/articubot_two/T1.dae" scale="1 1 1"/>
       </geometry>
     </collision>
@@ -63,9 +80,9 @@
     <material>Gazebo/White</material>
     </gazebo>
-  <!-- Joint between link_0 and base_link -->
-  <joint name="joint_1" type="revolute">
-    <parent link="base_link"/>
-    <child link="link_1"/>
-    <origin xyz="0.073 0.05597 0.02748" rpy="0 0 0"/>
+  <!-- Joint between link_1 and base_link -->
+  <joint name="joint_2" type="revolute">
+    <parent link="base_link"/>
+    <child link="link_2"/>
+    <origin xyz="-0.181 0.08 0.06" rpy="0 0 0"/>
     <axis xyz="1 0 0"/>
     <limit effort="5.0" velocity="1.0" lower="-0.540" upper="0.540"/>
@@ -75,10 +92,10 @@
     <visual>
       <geometry>
-        <mesh filename="/home/mikepzaza/Desktop/project2/src/articubot_two/T2V2.dae" scale="1 1 1"/>
-      </geometry>
-    </visual>
-    <collision>
-      <geometry>
-        <mesh filename="/home/mikepzaza/Desktop/project2/src/articubot_two/T2V2.dae" scale="1 1 1"/>
+        <mesh filename="file:///home/mikepzaza/Desktop/project2/src/articubot_two/T2V2.dae" scale="1 1 1"/>
+      </geometry>
+    </visual>
+    <collision>
+      <geometry>
+        <mesh filename="file:///home/mikepzaza/Desktop/project2/src/articubot_two/T2V2.dae" scale="1 1 1"/>
       </geometry>
     </collision>
@@ -90,11 +107,10 @@
     <material>Gazebo/White</material>
     </gazebo>
-  <!-- Joint between link_1 and base_link -->
-  <joint name="joint_2" type="revolute">
-    <parent link="base_link"/>
-    <child link="link_2"/>
-    <origin xyz="-0.278289 0.055976 0.02748" rpy="0 0 0"/>
-    <axis xyz="1 0 0"/>
-    <limit effort="5.0" velocity="1.0" lower="-0.540" upper="0.540"/>
+  <!-- Joint between link_0 and link_6 -->
+  <joint name="joint_6" type="continuous">
+    <parent link="base_link"/>
+    <child link="link_6"/>
+    <origin xyz="-0.215 -0.16 0" rpy="0 -${pi/2}  0"/>
+    <axis xyz="0 0 1"/>
   </joint>
   <!-- Link 6 (W1)-->
@@ -102,5 +118,5 @@
     <visual>
       <geometry>
-        <mesh filename="/home/mikepzaza/Desktop/project2/src/articubot_two/W1V2.dae" scale="1 1 1"/>
+        <cylinder radius="0.06" length="0.06"/>
       </geometry>
     </visual>
@@ -115,30 +131,4 @@
   </link>
     <gazebo reference="link_6">
-    <material>Gazebo/White</material>
-    </gazebo>
-  <!-- Joint between link_0 and link_6 -->
-  <joint name="joint_6" type="continuous">
-    <parent link="base_link"/>
-    <child link="link_6"/>
-    <origin xyz="-0.312 -0.214023 -0.03252" rpy="0 0 0"/>
-    <axis xyz="1 0 0"/>
-  </joint>
- <!-- Link 6 Clone (W3)-->
-  <link name="link_6_clone">
-    <visual>
-      <geometry>
-        <mesh filename="/home/mikepzaza/Desktop/project2/src/articubot_two/W1V2.dae" scale="1 1 1"/>
-      </geometry>
-    </visual>
-    <collision>
-      <geometry>
-          <cylinder radius="0.06" length="0.06"/>
-      </geometry>
-    </collision>
-    <xacro:inertial_cylinder mass="0.3" length="0.06" radius="0.06">
-        <origin xyz="0 0 0" rpy="0 0 0"/>
-    </xacro:inertial_cylinder>
-  </link>
-    <gazebo reference="link_6_clone">
     <material>Gazebo/White</material>
     </gazebo>
@@ -147,32 +137,58 @@
     <parent link="link_2"/>
     <child link="link_6_clone"/>
-    <origin xyz="-0.034 -0.07 -0.06" rpy="0 0 0"/>
-    <axis xyz="1 0 0"/>
-  </joint>
-  <!-- Link 6 Clone Clone (W5) -->
-  <link name="link_6_clone_clone">
-    <visual>
-      <geometry>
-        <mesh filename="/home/mikepzaza/Desktop/project2/src/articubot_two/W1V2.dae" scale="1 1 1"/>
-      </geometry>
-    </visual>
-    <collision>
-      <geometry>
-          <cylinder radius="0.06" length="0.06"/>
-      </geometry>
-    </collision>
-    <xacro:inertial_cylinder mass="0.3" length="0.06" radius="0.06">
-        <origin xyz="0 0 0" rpy="0 0 0"/>
-    </xacro:inertial_cylinder>
-  </link>
-    <gazebo reference="link_6_clone_clone">
-    <material>Gazebo/White</material>
-    </gazebo>
-  <!-- Joint between link_6_clone and link_6_clone_clone -->
+    <origin xyz="-0.035 -0.07 -0.06" rpy="0 1.57 0"/>
+    <axis xyz="0 0 1"/>
+  </joint>
+ <!-- Link 6 Clone (W3)-->
+  <link name="link_6_clone">
+    <visual>
+      <geometry>
+        <cylinder radius="0.06" length="0.06"/>
+      </geometry>
+    </visual>
+    <collision>
+      <geometry>
+          <cylinder radius="0.06" length="0.06"/>
+      </geometry>
+    </collision>
+    <xacro:inertial_cylinder mass="0.3" length="0.06" radius="0.06">
+        <origin xyz="0 0 0" rpy="0 0 0"/>
+    </xacro:inertial_cylinder>
+  </link>
+    <gazebo reference="link_6_clone">
+    <material>Gazebo/White</material>
+    </gazebo>
+  <!-- Joint between link_2 and link_6_clone_clone -->
   <joint name="joint_6_clone_clone" type="continuous">
     <parent link="link_2"/>
     <child link="link_6_clone_clone"/>
-    <origin xyz="-0.034 0.07 -0.06" rpy="0 0 0"/>
-    <axis xyz="1 0 0"/>
+    <origin xyz="-0.035 0.07 -0.06" rpy="0 1.57 0"/>
+    <axis xyz="0 0 1"/>
+  </joint>
+  <!-- Link 6 Clone Clone (W5) -->
+  <link name="link_6_clone_clone">
+    <visual>
+      <geometry>
+        <cylinder radius="0.06" length="0.06"/>
+      </geometry>
+    </visual>
+    <collision>
+      <geometry>
+          <cylinder radius="0.06" length="0.06"/>
+      </geometry>
+    </collision>
+    <xacro:inertial_cylinder mass="0.3" length="0.06" radius="0.06">
+        <origin xyz="0 0 0" rpy="0 0 0"/>
+    </xacro:inertial_cylinder>
+  </link>
+    <gazebo reference="link_6_clone_clone">
+    <material>Gazebo/White</material>
+    </gazebo>
+  <!-- Joint between base_link and link_7 -->
+  <joint name="joint_7" type="continuous">
+    <parent link="base_link"/>
+    <child link="link_7"/>
+    <origin xyz="0.205 -0.16 0" rpy="0 1.57 0"/>
+    <axis xyz="0 0 1"/>
   </joint>
   <!-- Link 7 (W2)-->
@@ -180,5 +196,5 @@
     <visual>
       <geometry>
-        <mesh filename="/home/mikepzaza/Desktop/project2/src/articubot_two/W2V2.dae" scale="1 1 1"/>
+        <cylinder radius="0.06" length="0.06"/>
       </geometry>
     </visual>
@@ -195,144 +211,55 @@
     <material>Gazebo/White</material>
     </gazebo>
-  <!-- Joint between base_link and link_7 -->
-  <joint name="joint_7" type="continuous">
-    <parent link="base_link"/>
-    <child link="link_7"/>
-    <origin xyz="0.106 -0.213773 -0.03252" rpy="0 0 0"/>
-    <axis xyz="1 0 0"/>
-  </joint>
-  <!-- Link 7 Clone (W4)-->
-  <link name="link_7_clone">
-    <visual>
-      <geometry>
-        <mesh filename="/home/mikepzaza/Desktop/project2/src/articubot_two/W2V2.dae" scale="1 1 1"/>
-      </geometry>
-    </visual>
-    <collision>
-      <geometry>
-          <cylinder radius="0.06" length="0.06"/>
-      </geometry>
-    </collision>
-    <xacro:inertial_cylinder mass="0.3" length="0.06" radius="0.06">
-        <origin xyz="0 0 0" rpy="0 0 0"/>
-    </xacro:inertial_cylinder>
-  </link>
-    <gazebo reference="link_7_clone">
-    <material>Gazebo/White</material>
-    </gazebo>
-  <!-- Joint between link_7 and link_7_clone -->
+  <!-- Joint between link_1 and link_7_clone -->
   <joint name="joint_7_clone" type="continuous">
     <parent link="link_1"/>
     <child link="link_7_clone"/>
-    <origin xyz="0.035 -0.07 -0.06" rpy="0 0 0"/>
-    <axis xyz="1 0 0"/>
-  </joint>
-  <!-- Link 7 Clone Clone (W6)-->
-  <link name="link_7_clone_clone">
-    <visual>
-      <geometry>
-        <mesh filename="/home/mikepzaza/Desktop/project2/src/articubot_two/W2V2.dae" scale="1 1 1"/>
-      </geometry>
-    </visual>
-    <collision>
-      <geometry>
-          <cylinder radius="0.06" length="0.06"/>
-      </geometry>
-    </collision>
-    <xacro:inertial_cylinder mass="0.3" length="0.06" radius="0.06">
-        <origin xyz="0 0 0" rpy="0 0 0"/>
-    </xacro:inertial_cylinder>
-  </link>
-    <gazebo reference="link_7_clone_clone">
-    <material>Gazebo/White</material>
-    </gazebo>
-  <!-- Joint between link_7_clone and link_7_clone_clone -->
+    <origin xyz="0.035 -0.07 -0.06" rpy="0 1.57 0"/>
+    <axis xyz="0 0 1"/>
+  </joint>
+  <!-- Link 7 Clone (W4)-->
+  <link name="link_7_clone">
+    <visual>
+      <geometry>
+        <cylinder radius="0.06" length="0.06"/>
+      </geometry>
+    </visual>
+    <collision>
+      <geometry>
+          <cylinder radius="0.06" length="0.06"/>
+      </geometry>
+    </collision>
+    <xacro:inertial_cylinder mass="0.3" length="0.06" radius="0.06">
+        <origin xyz="0 0 0" rpy="0 0 0"/>
+    </xacro:inertial_cylinder>
+  </link>
+    <gazebo reference="link_7_clone">
+    <material>Gazebo/White</material>
+    </gazebo>
+  <!-- Joint between link_1 and link_7_clone_clone -->
   <joint name="joint_7_clone_clone" type="continuous">
     <parent link="link_1"/>
     <child link="link_7_clone_clone"/>
-    <origin xyz="0.035 0.07 -0.06" rpy="0 0 0"/>
-    <axis xyz="1 0 0"/>
-  </joint>
- <!-- Link 8 (A1)-->
-  <link name="link_8">
-    <visual>
-      <geometry>
-        <mesh filename="/home/mikepzaza/Desktop/project2/src/articubot_two/A1V2.dae" scale="1 1 1"/>
-      </geometry>
-    </visual>
-    <collision>
-      <geometry>
-        <mesh filename="/home/mikepzaza/Desktop/project2/src/articubot_two/A1V2.dae" scale="1 1 1"/>
-      </geometry>
-    </collision>
-    <xacro:inertial_box mass="0.4" x="0.015" y="0.085" z="0.05">
-        <origin xyz="0 0 0" rpy="0 0 0"/>
-    </xacro:inertial_box>
-    </link>
-    <gazebo reference="link_8">
-    <material>Gazebo/White</material>
-    </gazebo>
-  <!-- Joint between link_0 and link_8 -->
-  <joint name="joint_8" type="revolute">
-    <parent link="base_link"/>
-    <child link="link_8"/>
-    <origin xyz="-0.247521 -0.078748 0.018452" rpy="0 0 0"/>
-    <axis xyz="1 0 0"/>
-    <limit effort="5.0" velocity="1.0" lower="-1.57" upper="1.57"/>
-  </joint>
-  <!-- Link 9 (A2)-->
-  <link name="link_9">
-    <visual>
-      <geometry>
-        <mesh filename="/home/mikepzaza/Desktop/project2/src/articubot_two/A2.dae" scale="1 1 1"/>
-      </geometry>
-    </visual>
-    <collision>
-      <geometry>
-        <mesh filename="/home/mikepzaza/Desktop/project2/src/articubot_two/A2.dae" scale="1 1 1"/>
-      </geometry>
-    </collision>
-    <xacro:inertial_box mass="0.3" x="0.015" y="0.180" z="0.1">
-        <origin xyz="0 0 0" rpy="0 0 0"/>
-    </xacro:inertial_box>
-  </link>
-    <gazebo reference="link_9">
-    <material>Gazebo/White</material>
-    </gazebo>
-  <!-- Joint between link_8 and link_9 -->
-  <joint name="joint_9" type="revolute">
-    <parent link="link_8"/>
-    <child link="link_9"/>
-    <origin xyz="0.015 -0.055 0" rpy="0 0 0"/>
-    <axis xyz="1 0 0"/>
-    <limit effort="5.0" velocity="1.0" lower="-1" upper="1.57"/>
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
Commit message: Update robot_core.xacro

File: robot_core.xacro (robot description, xacro)
@@ -2,18 +2,21 @@
 <robot xmlns:xacro="http://www.ros.org/wiki/xacro" >
 <xacro:include filename="inertial_macros.xacro" />
-    <material name="white">
-        <color rgba="1 1 1 1" />
-    </material>
-    <material name="orange">
-        <color rgba="1 0.3 0.1 1"/>
-    </material>
-    <material name="blue">
-        <color rgba="0.2 0.2 1 1"/>
-    </material>
-    <material name="black">
-        <color rgba="0 0 0 1"/>
-    </material>
+  <material name="white">
+    <color rgba="1 1 1 1" />
+  </material>
+  <material name="orange">
+    <color rgba="1 0.3 0.1 1"/>
+  </material>
+  <material name="blue">
+    <color rgba="0.2 0.2 1 1"/>
+  </material>
+  <material name="black">
+    <color rgba="0 0 0 1"/>
+  </material>
  <material name="red">
-     <color rgba="1 0 0 1"/>
+    <color rgba="1 0 0 1"/>
+ </material>
+ <material name="grey">
+    <color rgba="0.5 0.5 0.5 1"/>
  </material>
   <!-- BASE LINK -->
@@ -111,5 +114,5 @@
     <parent link="base_link"/>
     <child link="link_6"/>
-    <origin xyz="-0.215 -0.16 0" rpy="0 -${pi/2}  0"/>
+    <origin xyz="-0.215 -0.16 0" rpy="0 0 0"/>
     <axis xyz="0 0 1"/>
   </joint>
@@ -118,10 +121,10 @@
     <visual>
       <geometry>
-        <cylinder radius="0.06" length="0.06"/>
-      </geometry>
-    </visual>
-    <collision>
-      <geometry>
-        <cylinder radius="0.06" length="0.06"/>
+        <mesh filename="file:///home/mikepzaza/Desktop/project2/src/articubot_two/WV3.dae" scale="1 1 1"/>
+      </geometry>
+    </visual>
+    <collision>
+      <geometry>
+        <mesh filename="file:///home/mikepzaza/Desktop/project2/src/articubot_two/WV3.dae" scale="1 1 1"/>
       </geometry>
     </collision>
@@ -131,5 +134,5 @@
   </link>
     <gazebo reference="link_6">
-    <material>Gazebo/White</material>
+    <material>Gazebo/Grey</material>
     </gazebo>
   <!-- Joint between base_link and link_6_clone -->
@@ -137,5 +140,5 @@
     <parent link="link_2"/>
     <child link="link_6_clone"/>
-    <origin xyz="-0.035 -0.07 -0.06" rpy="0 1.57 0"/>
+    <origin xyz="-0.035 -0.07 -0.06" rpy="0 0 0"/>
     <axis xyz="0 0 1"/>
   </joint>
@@ -144,10 +147,10 @@
     <visual>
       <geometry>
-        <cylinder radius="0.06" length="0.06"/>
-      </geometry>
-    </visual>
-    <collision>
-      <geometry>
-          <cylinder radius="0.06" length="0.06"/>
+        <mesh filename="file:///home/mikepzaza/Desktop/project2/src/articubot_two/WV3.dae" scale="1 1 1"/>
+      </geometry>
+    </visual>
+    <collision>
+      <geometry>
+        <mesh filename="file:///home/mikepzaza/Desktop/project2/src/articubot_two/WV3.dae" scale="1 1 1"/>
       </geometry>
     </collision>
@@ -157,5 +160,5 @@
   </link>
     <gazebo reference="link_6_clone">
-    <material>Gazebo/White</material>
+    <material>Gazebo/Grey</material>
     </gazebo>
   <!-- Joint between link_2 and link_6_clone_clone -->
@@ -163,5 +166,5 @@
     <parent link="link_2"/>
     <child link="link_6_clone_clone"/>
-    <origin xyz="-0.035 0.07 -0.06" rpy="0 1.57 0"/>
+    <origin xyz="-0.035 0.07 -0.06" rpy="0 0 0"/>
     <axis xyz="0 0 1"/>
   </joint>
@@ -170,10 +173,10 @@
     <visual>
       <geometry>
-        <cylinder radius="0.06" length="0.06"/>
-      </geometry>
-    </visual>
-    <collision>
-      <geometry>
-          <cylinder radius="0.06" length="0.06"/>
+        <mesh filename="file:///home/mikepzaza/Desktop/project2/src/articubot_two/WV3.dae" scale="1 1 1"/>
+      </geometry>
+    </visual>
+    <collision>
+      <geometry>
+        <mesh filename="file:///home/mikepzaza/Desktop/project2/src/articubot_two/WV3.dae" scale="1 1 1"/>
       </geometry>
     </collision>
@@ -183,5 +186,5 @@
   </link>
     <gazebo reference="link_6_clone_clone">
-    <material>Gazebo/White</material>
+    <material>Gazebo/Grey</material>
     </gazebo>
   <!-- Joint between base_link and link_7 -->
@@ -189,5 +192,5 @@
     <parent link="base_link"/>
     <child link="link_7"/>
-    <origin xyz="0.205 -0.16 0" rpy="0 1.57 0"/>
+    <origin xyz="0.205 -0.16 0" rpy="0 0 0"/>
     <axis xyz="0 0 1"/>
   </joint>
@@ -196,10 +199,10 @@
     <visual>
       <geometry>
-        <cylinder radius="0.06" length="0.06"/>
-      </geometry>
-    </visual>
-    <collision>
-      <geometry>
-          <cylinder radius="0.06" length="0.06"/>
+        <mesh filename="file:///home/mikepzaza/Desktop/project2/src/articubot_two/WV3.dae" scale="1 1 1"/>
+      </geometry>
+    </visual>
+    <collision>
+      <geometry>
+        <mesh filename="file:///home/mikepzaza/Desktop/project2/src/articubot_two/WV3.dae" scale="1 1 1"/>
       </geometry>
     </collision>
@@ -209,5 +212,5 @@
   </link>
     <gazebo reference="link_7">
-    <material>Gazebo/White</material>
+    <material>Gazebo/Grey</material>
     </gazebo>
   <!-- Joint between link_1 and link_7_clone -->
@@ -215,5 +218,5 @@
     <parent link="link_1"/>
     <child link="link_7_clone"/>
-    <origin xyz="0.035 -0.07 -0.06" rpy="0 1.57 0"/>
+    <origin xyz="0.035 -0.07 -0.06" rpy="0 0 0"/>
     <axis xyz="0 0 1"/>
   </joint>
@@ -222,10 +225,10 @@
     <visual>
       <geometry>
-        <cylinder radius="0.06" length="0.06"/>
-      </geometry>
-    </visual>
-    <collision>
-      <geometry>
-          <cylinder radius="0.06" length="0.06"/>
+        <mesh filename="file:///home/mikepzaza/Desktop/project2/src/articubot_two/WV3.dae" scale="1 1 1"/>
+      </geometry>
+    </visual>
+    <collision>
+      <geometry>
+        <mesh filename="file:///home/mikepzaza/Desktop/project2/src/articubot_two/WV3.dae" scale="1 1 1"/>
       </geometry>
     </collision>
@@ -235,5 +238,5 @@
   </link>
     <gazebo reference="link_7_clone">
-    <material>Gazebo/White</material>
+    <material>Gazebo/Grey</material>
     </gazebo>
   <!-- Joint between link_1 and link_7_clone_clone -->
@@ -241,5 +244,5 @@
     <parent link="link_1"/>
     <child link="link_7_clone_clone"/>
-    <origin xyz="0.035 0.07 -0.06" rpy="0 1.57 0"/>
+    <origin xyz="0.035 0.07 -0.06" rpy="0 0 0"/>
     <axis xyz="0 0 1"/>
   </joint>
@@ -248,10 +251,10 @@
     <visual>
       <geometry>
-        <cylinder radius="0.06" length="0.06"/>
-      </geometry>
-    </visual>
-    <collision>
-      <geometry>
-          <cylinder radius="0.06" length="0.06"/>
+        <mesh filename="file:///home/mikepzaza/Desktop/project2/src/articubot_two/WV3.dae" scale="1 1 1"/>
+      </geometry>
+    </visual>
+    <collision>
+      <geometry>
+        <mesh filename="file:///home/mikepzaza/Desktop/project2/src/articubot_two/WV3.dae" scale="1 1 1"/>
       </geometry>
     </collision>
@@ -261,5 +264,5 @@
   </link>
     <gazebo reference="link_7_clone_clone">
-    <material>Gazebo/White</material>
+    <material>Gazebo/Grey</material>
     </gazebo>
 </robot>

Commit message: Update robot_core.xacro

File: robot_core.xacro (robot description, xacro)
@@ -49,5 +49,5 @@
       </geometry>
     </collision>
-    <xacro:inertial_box mass="4" x="0.480" y="0.510" z="0.33">
+    <xacro:inertial_box mass="3" x="0.480" y="0.510" z="0.33">
         <origin xyz="0 0 0" rpy="0 0 0"/>
     </xacro:inertial_box>
@@ -57,10 +57,8 @@
     </gazebo>
   <!-- Joint between link_0 and base_link -->
-  <joint name="joint_1" type="revolute">
+  <joint name="joint_1" type="fixed">
     <parent link="base_link"/>
     <child link="link_1"/>
     <origin xyz="0.170 0.08 0.06" rpy="0 0 0"/>
-    <axis xyz="1 0 0"/>
-    <limit effort="5.0" velocity="1.0" lower="-0.540" upper="0.540"/>
   </joint>
   <!-- Link 1 (T1)-->
@@ -84,10 +82,8 @@
     </gazebo>
   <!-- Joint between link_1 and base_link -->
-  <joint name="joint_2" type="revolute">
+  <joint name="joint_2" type="fixed">
     <parent link="base_link"/>
     <child link="link_2"/>
     <origin xyz="-0.181 0.08 0.06" rpy="0 0 0"/>
-    <axis xyz="1 0 0"/>
-    <limit effort="5.0" velocity="1.0" lower="-0.540" upper="0.540"/>
   </joint>
   <!-- Link 2 (T2)-->
@@ -115,5 +111,5 @@
     <child link="link_6"/>
     <origin xyz="-0.215 -0.16 0" rpy="0 0 0"/>
-    <axis xyz="0 0 1"/>
+    <axis xyz="1 0 0"/>
   </joint>
   <!-- Link 6 (W1)-->
@@ -141,5 +137,5 @@
     <child link="link_6_clone"/>
     <origin xyz="-0.035 -0.07 -0.06" rpy="0 0 0"/>
-    <axis xyz="0 0 1"/>
+    <axis xyz="1 0 0"/>
   </joint>
  <!-- Link 6 Clone (W3)-->
@@ -167,5 +163,5 @@
     <child link="link_6_clone_clone"/>
     <origin xyz="-0.035 0.07 -0.06" rpy="0 0 0"/>
-    <axis xyz="0 0 1"/>
+    <axis xyz="1 0 0"/>
   </joint>
   <!-- Link 6 Clone Clone (W5) -->
@@ -193,5 +189,5 @@
     <child link="link_7"/>
     <origin xyz="0.205 -0.16 0" rpy="0 0 0"/>
-    <axis xyz="0 0 1"/>
+    <axis xyz="1 0 0"/>
   </joint>
   <!-- Link 7 (W2)-->
@@ -219,5 +215,5 @@
     <child link="link_7_clone"/>
     <origin xyz="0.035 -0.07 -0.06" rpy="0 0 0"/>
-    <axis xyz="0 0 1"/>
+    <axis xyz="1 0 0"/>
   </joint>
   <!-- Link 7 Clone (W4)-->
@@ -245,5 +241,5 @@
     <child link="link_7_clone_clone"/>
     <origin xyz="0.035 0.07 -0.06" rpy="0 0 0"/>
-    <axis xyz="0 0 1"/>
+    <axis xyz="1 0 0"/>
   </joint>
   <!-- Link 7 Clone Clone (W6)-->
