Commit message: Update robot_core.xacro

File: robot_core.xacro (robot description, xacro)
@@ -20,4 +20,7 @@
     <color rgba="0.5 0.5 0.5 1"/>
  </material>
+ <material name="yellow">
+    <color rgba="1 1 0 1"/>  <!-- สีเหลือง -->
+ </material>
   <!-- BASE LINK -->
   <link name="base_link">
@@ -43,4 +46,5 @@
         <mesh filename="file:///home/mikepzaza/Desktop/project2/src/articubot_two/baselink.dae" scale="1 1 1"/>
       </geometry>
+      <material name="orange"/>
     </visual>
     <collision>
@@ -54,5 +58,83 @@
   </link>
     <gazebo reference="link_0">
-    <material>Gazebo/White</material>
+    <material>Gazebo/Orange</material>
+    </gazebo>
+  <!-- Joint between base_link and prop  -->
+  <joint name="joint_03" type="fixed">
+    <parent link="base_link"/>
+    <child link="link_03"/>
+    <origin xyz="-0.0025 0.155 0.17" rpy="0 0 0"/>
+  </joint>
+  <!-- Link 0(prop) -->
+  <link name="link_03">
+    <visual>
+      <geometry>
+        <mesh filename="file:///home/mikepzaza/Desktop/project2/src/articubot_two/prop.dae" scale="1 1 1"/>
+      </geometry>
+      <material name="blue"/>
+    </visual>
+    <collision>
+      <geometry>
+        <mesh filename="file:///home/mikepzaza/Desktop/project2/src/articubot_two/prop.dae" scale="1 1 1"/>
+      </geometry>
+    </collision>
+    <xacro:inertial_box mass="0.2" x="0.369" y="0.105" z="0.404">
+        <origin xyz="0 0 0" rpy="0 0 0"/>
+    </xacro:inertial_box>
+  </link>
+    <gazebo reference="link_03">
+    <material>Gazebo/Blue</material>
+    </gazebo>
+  <!-- Joint between link_0 and lackback -->
+  <joint name="joint_01" type="fixed">
+    <parent link="link_0"/>
+    <child link="link_01"/>
+    <origin xyz="-0.00552 0.265 0" rpy="0 0 1.57"/>
+  </joint>
+ <!-- Link_01 (lackback)-->
+  <link name="link_01">
+    <visual>
+      <geometry>
+        <mesh filename="file:///home/mikepzaza/Desktop/project2/src/articubot_two/lackback.dae" scale="1 1 1"/>
+      </geometry>
+      <material name="black"/>
+    </visual>
+    <collision>
+      <geometry>
+        <mesh filename="file:///home/mikepzaza/Desktop/project2/src/articubot_two/lackback.dae" scale="1 1 1"/>
+      </geometry>
+    </collision>
+    <xacro:inertial_box mass="0.1" x="0.48" y="0.005" z="0.17">
+        <origin xyz="0 0 0" rpy="0 0 0"/>
+    </xacro:inertial_box>
+  </link>
+    <gazebo reference="link_01">
+    <material>Gazebo/Black</material>
+    </gazebo>
+    <!-- Joint between link_0 and LED -->
+  <joint name="joint_02" type="fixed">
+    <parent link="link_0"/>
+    <child link="link_02"/>
+    <origin xyz="-0.00552 0.265 0.145" rpy="0 0 1.57"/>
+  </joint>
+ <!-- Link_01 (LED)-->
+  <link name="link_02">
+    <visual>
+      <geometry>
+        <mesh filename="file:///home/mikepzaza/Desktop/project2/src/articubot_two/LED.dae" scale="1 1 1"/>
+      </geometry>
+      <material name="red"/>
+    </visual>
+    <collision>
+      <geometry>
+        <mesh filename="file:///home/mikepzaza/Desktop/project2/src/articubot_two/LED.dae" scale="1 1 1"/>
+      </geometry>
+    </collision>
+    <xacro:inertial_box mass="0.03" x="0.45" y="0.005" z="0.03">
+        <origin xyz="0 0 0" rpy="0 0 0"/>
+    </xacro:inertial_box>
+  </link>
+    <gazebo reference="link_02">
+    <material>Gazebo/Red</material>
     </gazebo>
   <!-- Joint between link_0 and base_link -->
@@ -68,4 +150,5 @@
         <mesh filename="file:///home/mikepzaza/Desktop/project2/src/articubot_two/T1V2.dae" scale="1 1 1"/>
       </geometry>
+      <material name="blue"/>
     </visual>
     <collision>
@@ -79,5 +162,5 @@
   </link>
     <gazebo reference="link_1">
-    <material>Gazebo/White</material>
+    <material>Gazebo/Blue</material>
     </gazebo>
   <!-- Joint between link_1 and base_link -->
@@ -93,4 +176,5 @@
         <mesh filename="file:///home/mikepzaza/Desktop/project2/src/articubot_two/T2V2.dae" scale="1 1 1"/>
       </geometry>
+      <material name="blue"/>
     </visual>
     <collision>
@@ -104,5 +188,5 @@
   </link>
     <gazebo reference="link_2">
-    <material>Gazebo/White</material>
+    <material>Gazebo/Blue</material>
     </gazebo>
   <!-- Joint between link_0 and link_6 -->
@@ -119,4 +203,5 @@
         <mesh filename="file:///home/mikepzaza/Desktop/project2/src/articubot_two/WV3.dae" scale="1 1 1"/>
       </geometry>
+      <material name="grey"/>
     </visual>
     <collision>
@@ -145,4 +230,5 @@
         <mesh filename="file:///home/mikepzaza/Desktop/project2/src/articubot_two/WV3.dae" scale="1 1 1"/>
       </geometry>
+      <material name="grey"/>
     </visual>
     <collision>
@@ -171,4 +257,5 @@
         <mesh filename="file:///home/mikepzaza/Desktop/project2/src/articubot_two/WV3.dae" scale="1 1 1"/>
       </geometry>
+      <material name="grey"/>
     </visual>
     <collision>
@@ -197,4 +284,5 @@
         <mesh filename="file:///home/mikepzaza/Desktop/project2/src/articubot_two/WV3.dae" scale="1 1 1"/>
       </geometry>
+      <material name="grey"/>
     </visual>
     <collision>
@@ -223,4 +311,5 @@
         <mesh filename="file:///home/mikepzaza/Desktop/project2/src/articubot_two/WV3.dae" scale="1 1 1"/>
       </geometry>
+      <material name="grey"/>
     </visual>
     <collision>
@@ -249,4 +338,5 @@
         <mesh filename="file:///home/mikepzaza/Desktop/project2/src/articubot_two/WV3.dae" scale="1 1 1"/>
       </geometry>
+      <material name="grey"/>
     </visual>
     <collision>

Commit message: Update robot_core.xacro

File: robot_core.xacro (robot description, xacro)
@@ -150,5 +150,5 @@
         <mesh filename="file:///home/mikepzaza/Desktop/project2/src/articubot_two/T1V2.dae" scale="1 1 1"/>
       </geometry>
-      <material name="blue"/>
+      <material name="black"/>
     </visual>
     <collision>
@@ -162,5 +162,5 @@
   </link>
     <gazebo reference="link_1">
-    <material>Gazebo/Blue</material>
+    <material>Gazebo/Black</material>
     </gazebo>
   <!-- Joint between link_1 and base_link -->
@@ -176,5 +176,5 @@
         <mesh filename="file:///home/mikepzaza/Desktop/project2/src/articubot_two/T2V2.dae" scale="1 1 1"/>
       </geometry>
-      <material name="blue"/>
+      <material name="black"/>
     </visual>
     <collision>
@@ -188,5 +188,5 @@
   </link>
     <gazebo reference="link_2">
-    <material>Gazebo/Blue</material>
+    <material>Gazebo/Black</material>
     </gazebo>
   <!-- Joint between link_0 and link_6 -->

Commit message: Update robot_core.xacro

File: robot_core.xacro (robot description, xacro)
@@ -203,5 +203,4 @@
         <mesh filename="file:///home/mikepzaza/Desktop/project2/src/articubot_two/WV3.dae" scale="1 1 1"/>
       </geometry>
-      <material name="grey"/>
     </visual>
     <collision>
@@ -230,5 +229,4 @@
         <mesh filename="file:///home/mikepzaza/Desktop/project2/src/articubot_two/WV3.dae" scale="1 1 1"/>
       </geometry>
-      <material name="grey"/>
     </visual>
     <collision>
@@ -257,5 +255,4 @@
         <mesh filename="file:///home/mikepzaza/Desktop/project2/src/articubot_two/WV3.dae" scale="1 1 1"/>
       </geometry>
-      <material name="grey"/>
     </visual>
     <collision>
@@ -284,5 +281,4 @@
         <mesh filename="file:///home/mikepzaza/Desktop/project2/src/articubot_two/WV3.dae" scale="1 1 1"/>
       </geometry>
-      <material name="grey"/>
     </visual>
     <collision>
@@ -311,5 +307,4 @@
         <mesh filename="file:///home/mikepzaza/Desktop/project2/src/articubot_two/WV3.dae" scale="1 1 1"/>
       </geometry>
-      <material name="grey"/>
     </visual>
     <collision>
@@ -338,5 +333,4 @@
         <mesh filename="file:///home/mikepzaza/Desktop/project2/src/articubot_two/WV3.dae" scale="1 1 1"/>
       </geometry>
-      <material name="grey"/>
     </visual>
     <collision>
